Commit message: Disable front wheel drive

File: streetdrone_model/sd_description/urdf/wheels/sd_twizy_suspension.urdf.xacro (robot description, xacro)
@@ -163,13 +163,4 @@
             </actuator>
         </transmission>
-        <transmission name="front_left_rear_axle_trans">
-            <type>transmission_interface/SimpleTransmission</type>
-            <joint name="front_left_wheel_joint">
-                <hardwareInterface>hardware_interface/VelocityJointInterface</hardwareInterface>
-            </joint>
-            <actuator name="front_left_rear_axle_act">
-                <mechanicalReduction>1</mechanicalReduction>
-            </actuator>
-        </transmission>
     </xacro:macro>
     <xacro:macro name="FR_wheel">
@@ -196,13 +187,4 @@
             </actuator>
         </transmission>
-        <transmission name="front_right_rear_axle_trans">
-            <type>transmission_interface/SimpleTransmission</type>
-            <joint name="front_right_wheel_joint">
-                <hardwareInterface>hardware_interface/VelocityJointInterface</hardwareInterface>
-            </joint>
-            <actuator name="front_right_rear_axle_act">
-                <mechanicalReduction>1</mechanicalReduction>
-            </actuator>
-        </transmission>
     </xacro:macro>
     <xacro:macro name="RL_wheel">
