Commit message: Teleop node to drive SD model with a joystick

File: streetdrone_model/sd_description/urdf/sd_twizy.urdf.xacro (robot description, xacro)
@@ -65,7 +65,8 @@
       <fr_wheel_steering_d_gain>3e2</fr_wheel_steering_d_gain>
       <max_speed>22</max_speed>
-      <max_torque>526</max_torque>
-      <front_brake_torque>526</front_brake_torque>
-      <back_brake_torque>526</back_brake_torque>
+      <max_torque>250</max_torque>
+      <front_brake_torque>260</front_brake_torque>
+      <back_brake_torque>260</back_brake_torque>
+      <chassis_aero_force_gain>0.63045</chassis_aero_force_gain>
     </plugin>
   </gazebo>

File: streetdrone_model/sd_description/urdf/wheels/sd_twizy_suspension.urdf.xacro (robot description, xacro)
@@ -12,5 +12,5 @@
   <xacro:property name = "front_wheel_mass" value="9.14"/>
   <xacro:property name = "front_tyre_width" value="0.125"/>
-  <xacro:property name = "friction_dry_mu" value="0.85"/>
+  <xacro:property name = "friction_dry_mu" value="0.95"/>
   <xacro:property name = "friction_wet_mu" value="0.4"/>
   <xacro:property name = "degrees_90" value="1.57079633"/>
