Commit message: Updated sensors, vehicle controls and worlds

File: streetdrone_model/sd_description/urdf/sd_twizy.urdf (robot description, URDF)
Before this commit: robot sd_twizy, 26 links, 25 joints
Links:
- link base_link: geometry collision mesh filename=file:////home/efimiap2/catkin_ws/src/streetdrone_model/sd_d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 scale=0.01 0.01 0.01; visual mesh filename=file:////home/efimiap2/catkin_ws/src/streetdrone_model/sd_d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 scale=0.01 0.01 0.01
- link velodyne: geometry visual mesh filename=file:////home/efimiap2/catkin_ws/src/streetdrone_model/sd_d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
- link velodyne_base_link: geometry collision cylinder length=0.0717 radius=0.0516; visual mesh filename=file:////home/efimiap2/catkin_ws/src/streetdrone_model/sd_d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
Joints:
- joint vehicle_base_joint: origin xyz=0 0 0 rpy=0 0 0 -> xyz=0 0 0.281 rpy=0 0 0

File: streetdrone_model/sd_description/urdf/sd_twizy.urdf.xacro (robot description, xacro)
@@ -26,27 +26,27 @@
         <origin xyz="-0.681 0 1.445" rpy="0 -${1.5*M_PI/180.0} 0"/>
     </xacro:VLP-16>
-    <xacro:sekonix_camera frlr_prefix="front" lrc_prefix="left">
+    <xacro:blackfly_camera frlr_prefix="front" lrc_prefix="left">
         <origin xyz="-0.04 0.12 1.3" rpy="0 0.087 0"/>
-    </xacro:sekonix_camera>
-    <xacro:sekonix_camera frlr_prefix="front" lrc_prefix="right">
+    </xacro:blackfly_camera>
+    <xacro:blackfly_camera frlr_prefix="front" lrc_prefix="right">
         <origin xyz="-0.04 -0.12 1.3" rpy="0 0.087 0"/>
-    </xacro:sekonix_camera>
-    <xacro:sekonix_camera frlr_prefix="front" lrc_prefix="center">
+    </xacro:blackfly_camera>
+    <xacro:blackfly_camera frlr_prefix="front" lrc_prefix="center">
         <origin xyz="-0.04 0 1.3" rpy="0 0.087 0"/>
-    </xacro:sekonix_camera>
-    <xacro:sekonix_camera frlr_prefix="rear" lrc_prefix="center">
+    </xacro:blackfly_camera>
+    <xacro:blackfly_camera frlr_prefix="rear" lrc_prefix="center">
         <origin xyz="-1.26 0 1.28" rpy="0 0.2618 3.14"/>
-    </xacro:sekonix_camera>
-    <xacro:sekonix_camera frlr_prefix="right" lrc_prefix="forward">
+    </xacro:blackfly_camera>
+    <xacro:blackfly_camera frlr_prefix="right" lrc_prefix="forward">
         <origin xyz="-0.95 -0.42 1.2" rpy="0 0.244 -1.12"/>
-    </xacro:sekonix_camera>
-    <xacro:sekonix_camera frlr_prefix="right" lrc_prefix="rearward">
+    </xacro:blackfly_camera>
+    <xacro:blackfly_camera frlr_prefix="right" lrc_prefix="rearward">
         <origin xyz="-1.05 -0.42 1.2" rpy="0 0.244 -2.18"/>
-    </xacro:sekonix_camera>
-    <xacro:sekonix_camera frlr_prefix="left" lrc_prefix="forward">
+    </xacro:blackfly_camera>
+    <xacro:blackfly_camera frlr_prefix="left" lrc_prefix="forward">
         <origin xyz="-0.95 0.4 1.2" rpy="0 0.2967 1.12"/>
-    </xacro:sekonix_camera>
-    <xacro:sekonix_camera frlr_prefix="left" lrc_prefix="rearward">
+    </xacro:blackfly_camera>
+    <xacro:blackfly_camera frlr_prefix="left" lrc_prefix="rearward">
         <origin xyz="-1.05 0.39 1.2" rpy="0 0.2967 2.18"/>
-    </xacro:sekonix_camera>
+    </xacro:blackfly_camera>
 </robot>

File: streetdrone_model/sd_description/urdf/sensors/cameras.urdf.xacro (robot description, xacro)
@@ -5,6 +5,6 @@
   All rights reserved
 -->
-<robot xmlns:xacro="http://www.ros.org/wiki/xacro" name="sekonix_camera">
-    <xacro:macro name="sekonix_camera" params="frlr_prefix lrc_prefix *origin">
+<robot xmlns:xacro="http://www.ros.org/wiki/xacro" name="blackfly_camera">
+    <xacro:macro name="blackfly_camera" params="frlr_prefix lrc_prefix *origin">
         <joint name="${frlr_prefix}_${lrc_prefix}_camera_joint" type="fixed">
             <axis xyz="0 1 0" />
@@ -53,6 +53,6 @@
                     <horizontal_fov>2.09</horizontal_fov>
                     <image>
-                        <width>1928</width>
-                        <height>1208</height>
+                        <width>1920</width>
+                        <height>1200</height>
                         <format>R8G8B8</format>
                     </image>

File: streetdrone_model/sd_description/urdf/wheels/sd_twizy_suspension.urdf.xacro (robot description, xacro)
@@ -12,5 +12,5 @@
     <xacro:property name = "front_wheel_mass" value="9.14"/>
     <xacro:property name = "front_tyre_width" value="0.125"/>
-    <xacro:property name = "friction_dry_mu" value="0.85"/>
+    <xacro:property name = "friction_dry_mu" value="1"/>
     <xacro:property name = "friction_wet_mu" value="0.4"/>
     <xacro:property name = "degrees_90" value="1.57079633"/>

Commit message: Version 2.1.0 ROS Kinetic
* Updated sensors, vehicle controls and worlds

* Version 2.1.0 ROS Kinetic

* Cameras resolution

* Blackfly cameras tag

* Readme update

File: streetdrone_model/sd_description/urdf/sd_twizy.urdf (robot description, URDF)
Before this commit: robot sd_twizy, 26 links, 25 joints
Links:
- removed link vehicle_base
- added link chassis, mass 435; collision mesh filename=file:////home/efimiap2/catkin_ws/src/streetdrone_model/sd_d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 scale=0.01 0.01 0.01; visual mesh filename=file:////home/efimiap2/catkin_ws/src/streetdrone_model/sd_d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 scale=0.01 0.01 0.01
- link base_link: mass 435 -> None; geometry visual box size=0.001 0.001 0.001
Joints:
- removed joint vehicle_base_joint
- added joint chassis_joint: type fixed, parent base_link, child chassis, origin xyz=0.843 0 0 rpy=0 0 0
- joint front_center_camera_joint: parent base_link -> chassis
- joint front_left_camera_joint: parent base_link -> chassis
- joint front_left_steer_joint: origin xyz=0.843 -0.54 0 rpy=1.57079633 0 3.14159265 -> xyz=1.686 -0.54 0 rpy=1.57079633 0 3.14159265
- joint front_right_camera_joint: parent base_link -> chassis
- joint front_right_steer_joint: origin xyz=0.843 0.54 0 rpy=1.57079633 0 3.14159265 -> xyz=1.686 0.54 0 rpy=1.57079633 0 3.14159265
- joint left_forward_camera_joint: parent base_link -> chassis
- joint left_rearward_camera_joint: parent base_link -> chassis
- joint rear_center_camera_joint: parent base_link -> chassis
- joint rear_left_wheel_joint: origin xyz=-0.843 -0.54 0 rpy=1.57079633 0 3.14159265 -> xyz=0 -0.54 0 rpy=1.57079633 0 0
- joint rear_right_wheel_joint: origin xyz=-0.843 0.54 0 rpy=1.57079633 0 3.14159265 -> xyz=0 0.54 0 rpy=1.57079633 0 0
- joint right_forward_camera_joint: parent base_link -> chassis
- joint right_rearward_camera_joint: parent base_link -> chassis
- joint velodyne_base_mount_joint: parent base_link -> chassis

File: streetdrone_model/sd_description/urdf/sensors/cameras.urdf.xacro (robot description, xacro)
@@ -1,47 +1,47 @@
 <?xml version="1.0"?>
 <!--
-  Copyright (c) 2019 StreetDrone Limited
-  Author:  Efimia Panagiotaki
-  All rights reserved
+Copyright (c) 2020 StreetDrone Limited
+Author:  Efimia Panagiotaki
+All rights reserved
 -->
 <robot xmlns:xacro="http://www.ros.org/wiki/xacro" name="blackfly_camera">
     <xacro:macro name="blackfly_camera" params="frlr_prefix lrc_prefix *origin">
-        <joint name="${frlr_prefix}_${lrc_prefix}_camera_joint" type="fixed">
-            <axis xyz="0 1 0" />
-            <xacro:insert_block name="origin"/>
-            <parent link="base_link"/>
-            <child link="${frlr_prefix}_${lrc_prefix}_camera_link"/>
-        </joint>
-        <!-- Camera -->
-        <link name="${frlr_prefix}_${lrc_prefix}_camera_link">
-            <collision>
-                <origin xyz="0 0 0" rpy="0 0 0"/>
-                <geometry>
-                    <box size="0.026 0.026 0.0203"/>
-                </geometry>
-            </collision>
-            <visual>
-                <origin xyz="0 0 0" rpy="0 0 0"/>
-                <geometry>
-                    <box size="0.026 0.026 0.0203"/>
-                </geometry>
-                <material name="red"/>
-            </visual>
-            <inertial>
-                <mass value="1e-5" />
-                <origin xyz="0 0 0" rpy="0 0 0"/>
-                <inertia ixx="1e-6" ixy="0" ixz="0" iyy="1e-6" iyz="0" izz="1e-6" />
-            </inertial>
-        </link>
-        <!-- generate an optical frame http://www.ros.org/reps/rep-0103.html#suffix-frames
-            so that ros and opencv can operate on the camera frame correctly -->
-        <joint name="${frlr_prefix}_${lrc_prefix}_camera_optical_joint" type="fixed">
-            <!-- these values have to be these values otherwise the gazebo camera image
-                won't be aligned properly with the frame it is supposedly originating from -->
-            <origin xyz="0 0 0" rpy="${-pi/2} 0 ${-pi/2}"/>
-            <parent link="${frlr_prefix}_${lrc_prefix}_camera_link"/>
-            <child link="${frlr_prefix}_${lrc_prefix}_camera_link_optical"/>
-        </joint>
-        <link name="${frlr_prefix}_${lrc_prefix}_camera_link_optical"/>
+    <joint name="${frlr_prefix}_${lrc_prefix}_camera_joint" type="fixed">
+      <axis xyz="0 1 0" />
+      <xacro:insert_block name="origin"/>
+      <parent link="chassis"/>
+      <child link="${frlr_prefix}_${lrc_prefix}_camera_link"/>
+    </joint>
+    <!-- Camera -->
+    <link name="${frlr_prefix}_${lrc_prefix}_camera_link">
+      <collision>
+        <origin xyz="0 0 0" rpy="0 0 0"/>
+        <geometry>
+          <box size="0.026 0.026 0.0203"/>
+        </geometry>
+      </collision>
+      <visual>
+        <origin xyz="0 0 0" rpy="0 0 0"/>
+        <geometry>
+          <box size="0.026 0.026 0.0203"/>
+        </geometry>
+        <material name="red"/>
+      </visual>
+      <inertial>
+        <mass value="1e-5" />
+        <origin xyz="0 0 0" rpy="0 0 0"/>
+        <inertia ixx="1e-6" ixy="0" ixz="0" iyy="1e-6" iyz="0" izz="1e-6" />
+      </inertial>
+    </link>
+    <!-- generate an optical frame http://www.ros.org/reps/rep-0103.html#suffix-frames
+         so that ros and opencv can operate on the camera frame correctly -->
+    <joint name="${frlr_prefix}_${lrc_prefix}_camera_optical_joint" type="fixed">
+      <!-- these values have to be these values otherwise the gazebo camera image
+           won't be aligned properly with the frame it is supposedly originating from -->
+      <origin xyz="0 0 0" rpy="${-pi/2} 0 ${-pi/2}"/>
+      <parent link="${frlr_prefix}_${lrc_prefix}_camera_link"/>
+      <child link="${frlr_prefix}_${lrc_prefix}_camera_link_optical"/>
+    </joint>
+    <link name="${frlr_prefix}_${lrc_prefix}_camera_link_optical"/>
         <gazebo reference="${frlr_prefix}_${lrc_prefix}_camera_link">
             <mu1>0.2</mu1>
@@ -93,4 +93,4 @@
             </sensor>
         </gazebo>
-    </xacro:macro>
+  </xacro:macro>
 </robot>
