Commit message: Beta v0.2.0 of the SD Twizy Gazebo model
* Split the packages
* Added _description package containing the URDF and the meshes

File: streetdrone_model/sd_description/urdf/bases/sd_twizy_body.urdf.xacro (robot description, xacro)
@@ -6,5 +6,5 @@
 -->
 <robot name="sd_twizy" xmlns:xacro="http://www.ros.org/wiki/xacro">
-    <xacro:include filename="$(find sd_robot)/urdf/bases/sd_twizy_body.gazebo.xacro" />
+    <xacro:include filename="$(find sd_description)/urdf/bases/sd_twizy_body.gazebo.xacro" />
     <xacro:macro name="sd_twizy_base" params="name">
         <xacro:property name="depth" value="2.352"/>
@@ -35,5 +35,5 @@
                 <origin xyz="0 0 0" rpy="0 0 1.57"/>
                 <geometry>
-                    <mesh filename="file:///$(find sd_robot)/meshes/SDTwizy.stl" scale="0.01 0.01 0.01"/>
+                    <mesh filename="file:///$(find sd_description)/meshes/SDTwizy.stl" scale="0.01 0.01 0.01"/>
 		        </geometry>
             </visual>

File: streetdrone_model/sd_description/urdf/sd_twizy.urdf.xacro (robot description, xacro)
@@ -9,8 +9,8 @@
     <!-- Imported elements -->
     <!-- ***************** -->
-    <xacro:include filename="$(find sd_robot)/urdf/bases/sd_twizy_body.urdf.xacro" />
-    <xacro:include filename="$(find sd_robot)/urdf/wheels/sd_twizy_suspension.urdf.xacro" />
-    <xacro:include filename="$(find sd_robot)/urdf/sensors/VLP-16.urdf.xacro"/>
-    <xacro:include filename="$(find sd_robot)/urdf/sensors/cameras.urdf.xacro"/>
+    <xacro:include filename="$(find sd_description)/urdf/bases/sd_twizy_body.urdf.xacro" />
+    <xacro:include filename="$(find sd_description)/urdf/wheels/sd_twizy_suspension.urdf.xacro" />
+    <xacro:include filename="$(find sd_description)/urdf/sensors/VLP-16.urdf.xacro"/>
+    <xacro:include filename="$(find sd_description)/urdf/sensors/cameras.urdf.xacro"/>
     <!-- *************** -->
     <!-- Robots Elements -->

File: streetdrone_model/sd_description/urdf/sensors/VLP-16.urdf.xacro (robot description, xacro)
@@ -18,10 +18,10 @@
             <visual>
                 <geometry>
-                    <mesh filename="file:///$(find sd_robot)/meshes/VLP16_base_1.dae" />
+                    <mesh filename="file:///$(find sd_description)/meshes/VLP16_base_1.dae" />
                 </geometry>
             </visual>
             <visual>
                 <geometry>
-                    <mesh filename="file:///$(find sd_robot)/meshes/VLP16_base_2.dae" />
+                    <mesh filename="file:///$(find sd_description)/meshes/VLP16_base_2.dae" />
                 </geometry>
             </visual>
@@ -47,5 +47,5 @@
                 <origin xyz="0 0 -0.0377" />
                 <geometry>
-                    <mesh filename="file:///$(find sd_robot)/meshes/VLP16_scan.dae" />
+                    <mesh filename="file:///$(find sd_description)/meshes/VLP16_scan.dae" />
                 </geometry>
             </visual>

Commit message: Use STL mesh for body collision model
Uses a simplified convex hull of the visual mesh as the collision geometry

File: streetdrone_model/sd_description/urdf/bases/sd_twizy_body.urdf.xacro (robot description, xacro)
@@ -41,6 +41,6 @@
                 <origin xyz="0 0 ${clearance}" rpy="-0.0135 0 1.57"/>
                 <geometry>
-                    <box size="${width} ${depth} ${height}"/>
-                </geometry>
+                    <mesh filename="file:///$(find sd_description)/meshes/SDTwizy_collision.stl" scale="0.01 0.01 0.01"/>
+		</geometry>
             </collision>
         </link>

Commit message: Update clearance so car starts with rear wheels on the ground

File: streetdrone_model/sd_description/urdf/bases/sd_twizy_body.urdf.xacro (robot description, xacro)
@@ -12,5 +12,5 @@
         <xacro:property name="width" value="1.431"/>
         <xacro:property name="base_mass" value="435"/>
-        <xacro:property name="clearance" value="0.582"/>
+        <xacro:property name="clearance" value="0.281"/>
         <link name="vehicle_base">
             <visual>
@@ -22,5 +22,5 @@
         </link>
         <joint name="vehicle_base_joint" type="fixed">
-            <origin xyz="0 0 0" rpy="0 0 0"/>
+            <origin xyz="0 0 ${clearance}" rpy="0 0 0"/>
             <parent link="vehicle_base"/>
             <child link="base_link"/>
@@ -33,11 +33,11 @@
             </inertial>
             <visual>
-                <origin xyz="0 0 0" rpy="0 0 1.57"/>
+                <origin xyz="0 0 0" rpy="0 0 1.57079632679"/>
                 <geometry>
                     <mesh filename="file:///$(find sd_description)/meshes/SDTwizy.stl" scale="0.01 0.01 0.01"/>
-		        </geometry>
+		</geometry>
             </visual>
             <collision>
-                <origin xyz="0 0 ${clearance}" rpy="-0.0135 0 1.57"/>
+                <origin xyz="0 0 0" rpy="0 0 1.57079632679"/>
                 <geometry>
                     <mesh filename="file:///$(find sd_description)/meshes/SDTwizy_collision.stl" scale="0.01 0.01 0.01"/>

Commit message: Mesh and collision model fixes and updates (#2)
* Fix inverted faces in STL

Makes them visible from the correct viewing angle

* Use STL mesh for body collision model

Uses a simplified convex hull of the visual mesh as the collision geometry

* Update clearance so car starts with rear wheels on the ground

File: streetdrone_model/sd_description/urdf/bases/sd_twizy_body.urdf.xacro (robot description, xacro)
@@ -12,5 +12,5 @@
         <xacro:property name="width" value="1.431"/>
         <xacro:property name="base_mass" value="435"/>
-        <xacro:property name="clearance" value="0.582"/>
+        <xacro:property name="clearance" value="0.281"/>
         <link name="vehicle_base">
             <visual>
@@ -22,5 +22,5 @@
         </link>
         <joint name="vehicle_base_joint" type="fixed">
-            <origin xyz="0 0 0" rpy="0 0 0"/>
+            <origin xyz="0 0 ${clearance}" rpy="0 0 0"/>
             <parent link="vehicle_base"/>
             <child link="base_link"/>
@@ -33,14 +33,14 @@
             </inertial>
             <visual>
-                <origin xyz="0 0 0" rpy="0 0 1.57"/>
+                <origin xyz="0 0 0" rpy="0 0 1.57079632679"/>
                 <geometry>
                     <mesh filename="file:///$(find sd_description)/meshes/SDTwizy.stl" scale="0.01 0.01 0.01"/>
-		        </geometry>
+		</geometry>
             </visual>
             <collision>
-                <origin xyz="0 0 ${clearance}" rpy="-0.0135 0 1.57"/>
+                <origin xyz="0 0 0" rpy="0 0 1.57079632679"/>
                 <geometry>
-                    <box size="${width} ${depth} ${height}"/>
-                </geometry>
+                    <mesh filename="file:///$(find sd_description)/meshes/SDTwizy_collision.stl" scale="0.01 0.01 0.01"/>
+		</geometry>
             </collision>
         </link>

Commit message: Fix too many slashes in file paths

File: streetdrone_model/sd_description/urdf/bases/sd_twizy_body.urdf.xacro (robot description, xacro)
@@ -36,5 +36,5 @@
         <origin xyz="0 0 0" rpy="0 0 1.57079632679"/>
         <geometry>
-          <mesh filename="file:///$(find sd_description)/meshes/SDTwizy.stl" scale="0.01 0.01 0.01"/>
+          <mesh filename="file://$(find sd_description)/meshes/SDTwizy.stl" scale="0.01 0.01 0.01"/>
         </geometry>
       </visual>
@@ -42,5 +42,5 @@
         <origin xyz="0 0 0" rpy="0 0 1.57079632679"/>
         <geometry>
-          <mesh filename="file:///$(find sd_description)/meshes/SDTwizy_collision.stl" scale="0.01 0.01 0.01"/>
+          <mesh filename="file://$(find sd_description)/meshes/SDTwizy_collision.stl" scale="0.01 0.01 0.01"/>
         </geometry>
       </collision>

File: streetdrone_model/sd_description/urdf/sensors/VLP-16.urdf.xacro (robot description, xacro)
@@ -18,10 +18,10 @@
             <visual>
                 <geometry>
-                    <mesh filename="file:///$(find sd_description)/meshes/VLP16_base_1.dae" />
+                    <mesh filename="file://$(find sd_description)/meshes/VLP16_base_1.dae" />
                 </geometry>
             </visual>
             <visual>
                 <geometry>
-                    <mesh filename="file:///$(find sd_description)/meshes/VLP16_base_2.dae" />
+                    <mesh filename="file://$(find sd_description)/meshes/VLP16_base_2.dae" />
                 </geometry>
             </visual>
@@ -47,5 +47,5 @@
                 <origin xyz="0 0 -0.0377" />
                 <geometry>
-                    <mesh filename="file:///$(find sd_description)/meshes/VLP16_scan.dae" />
+                    <mesh filename="file://$(find sd_description)/meshes/VLP16_scan.dae" />
                 </geometry>
             </visual>
