Commit message: Cleanup URDF files and make links and joints resolvable in plugin

File: streetdrone_model/sd_description/urdf/bases/sd_twizy_body.gazebo.xacro (robot description, xacro)
@@ -1,7 +1,7 @@
 <?xml version="1.0"?>
 <!--
-  Copyright (c) 2019 StreetDrone Limited
-  Author:  Efimia Panagiotaki
-  All rights reserved
+Copyright (c) 2019 StreetDrone Limited
+Author:  Efimia Panagiotaki
+All rights reserved
 -->
 <robot xmlns:xacro="http://www.ros.org/wiki/xacro">
@@ -17,14 +17,14 @@
   <xacro:macro name="ros_control">
     <gazebo>
-            <plugin name="gazebo_ros_control" filename="libgazebo_ros_control.so">
-                <robotNamespace>/sd_twizy</robotNamespace>
-                <controlPeriod>0.001</controlPeriod>
-                <robotSimType>gazebo_ros_control/DefaultRobotHWSim</robotSimType>
-                <legacyModeNS>true</legacyModeNS>
-            </plugin>
-        </gazebo>
-    </xacro:macro>
-    <gazebo reference="base_link">-->
-        <material>Gazebo/Green</material>
+      <plugin name="gazebo_ros_control" filename="libgazebo_ros_control.so">
+        <robotNamespace>/sd_twizy</robotNamespace>
+        <controlPeriod>0.001</controlPeriod>
+        <robotSimType>gazebo_ros_control/DefaultRobotHWSim</robotSimType>
+        <legacyModeNS>true</legacyModeNS>
+      </plugin>
     </gazebo>
+  </xacro:macro>
+  <gazebo reference="chassis">
+    <material>Gazebo/Green</material>
+  </gazebo>
 </robot>

File: streetdrone_model/sd_description/urdf/bases/sd_twizy_body.urdf.xacro (robot description, xacro)
@@ -1,48 +1,49 @@
 <?xml version="1.0"?>
 <!--
-  Copyright (c) 2019 StreetDrone Limited
-  Author:  Efimia Panagiotaki
-  All rights reserved
+Copyright (c) 2019 StreetDrone Limited
+Author:  Efimia Panagiotaki
+All rights reserved
 -->
 <robot name="sd_twizy" xmlns:xacro="http://www.ros.org/wiki/xacro">
-    <xacro:include filename="$(find sd_description)/urdf/bases/sd_twizy_body.gazebo.xacro" />
-    <xacro:macro name="sd_twizy_base" params="name">
-        <xacro:property name="depth" value="2.352"/>
-        <xacro:property name="height" value="1.7"/>
-        <xacro:property name="width" value="1.431"/>
-        <xacro:property name="base_mass" value="435"/>
-        <xacro:property name="clearance" value="0.281"/>
-        <link name="vehicle_base">
-            <visual>
-                <origin xyz="0 0 0" rpy="0 0 0" />
-                <geometry>
-                    <box size="0.001 0.001 0.001" />
-                </geometry>
-            </visual>
-        </link>
-        <joint name="vehicle_base_joint" type="fixed">
-            <origin xyz="0 0 ${clearance}" rpy="0 0 0"/>
-            <parent link="vehicle_base"/>
-            <child link="base_link"/>
-        </joint>
-        <link name="base_link">
-            <inertial>
-                <mass value="${base_mass}"/>
-                <origin xyz="0 0 0"/>
-                <inertia ixx="243.175" ixy="0" ixz="0" iyy="430.166" iyz="0" izz="430.166"/>
-            </inertial>
-            <visual>
-                <origin xyz="0 0 0" rpy="0 0 1.57079632679"/>
-                <geometry>
-                    <mesh filename="file:///$(find sd_description)/meshes/SDTwizy.stl" scale="0.01 0.01 0.01"/>
-		</geometry>
-            </visual>
-            <collision>
-                <origin xyz="0 0 0" rpy="0 0 1.57079632679"/>
-                <geometry>
-                    <mesh filename="file:///$(find sd_description)/meshes/SDTwizy_collision.stl" scale="0.01 0.01 0.01"/>
-		</geometry>
-            </collision>
-        </link>
-    </xacro:macro>
+  <xacro:include filename="$(find sd_description)/urdf/bases/sd_twizy_body.gazebo.xacro" />
+  <xacro:macro name="sd_twizy_base" params="name">
+    <xacro:property name="depth" value="2.352"/>
+    <xacro:property name="height" value="1.7"/>
+    <xacro:property name="width" value="1.431"/>
+    <xacro:property name="base_mass" value="435"/>
+    <xacro:property name="clearance" value="0.281"/>
+    <xacro:property name = "wheelbase" value="1.686"/>
+    <link name="base_link">
+      <visual>
+        <origin xyz="0 0 0" rpy="0 0 0" />
+        <geometry>
+          <box size="0.001 0.001 0.001" />
+        </geometry>
+      </visual>
+    </link>
+    <joint name="chassis_joint" type="fixed">
+      <origin xyz="${wheelbase / 2} 0 0" rpy="0 0 0"/>
+      <parent link="base_link"/>
+      <child link="chassis"/>
+    </joint>
+    <link name="chassis">
+      <inertial>
+        <mass value="${base_mass}"/>
+        <origin xyz="0 0 0"/>
+        <inertia ixx="243.175" ixy="0" ixz="0" iyy="430.166" iyz="0" izz="430.166"/>
+      </inertial>
+      <visual>
+        <origin xyz="0 0 0" rpy="0 0 1.57079632679"/>
+        <geometry>
+          <mesh filename="file:///$(find sd_description)/meshes/SDTwizy.stl" scale="0.01 0.01 0.01"/>
+        </geometry>
+      </visual>
+      <collision>
+        <origin xyz="0 0 0" rpy="0 0 1.57079632679"/>
+        <geometry>
+          <mesh filename="file:///$(find sd_description)/meshes/SDTwizy_collision.stl" scale="0.01 0.01 0.01"/>
+        </geometry>
+      </collision>
+    </link>
+  </xacro:macro>
 </robot>

File: streetdrone_model/sd_description/urdf/sd_twizy.urdf.xacro (robot description, xacro)
@@ -1,56 +1,62 @@
 <?xml version="1.0"?>
 <!--
-  Copyright (c) 2019 StreetDrone Limited
-  Author:  Efimia Panagiotaki
-  All rights reserved
+Copyright (c) 2019 StreetDrone Limited
+Author:  Efimia Panagiotaki
+All rights reserved
 -->
 <robot name="sd_twizy" xmlns:xacro="http://www.ros.org/wiki/xacro">
+  <!-- ***************** -->
+  <!-- Imported elements -->
+  <!-- ***************** -->
+  <xacro:include filename="$(find sd_description)/urdf/bases/sd_twizy_body.urdf.xacro" />
+  <xacro:include filename="$(find sd_description)/urdf/wheels/sd_twizy_suspension.urdf.xacro" />
+  <xacro:include filename="$(find sd_description)/urdf/sensors/VLP-16.urdf.xacro"/>
+  <xacro:include filename="$(find sd_description)/urdf/sensors/cameras.urdf.xacro"/>
+  <!-- *************** -->
+  <!-- Robots Elements -->
+  <!-- *************** -->
+  <xacro:sd_twizy_base name="sd_twizy"/>
+  <xacro:RL_wheel/>
+  <xacro:RR_wheel/>
+  <xacro:FL_wheel/>
+  <xacro:FR_wheel/>
+  <!-- Sensors -->
+  <xacro:VLP-16  parent="chassis" name="velodyne" topic="/points_raw" hz="10" samples="1875">
+    <origin xyz="-0.681 0 1.445" rpy="0 -${1.5*M_PI/180.0} 0"/>
+  </xacro:VLP-16>
+  <xacro:sekonix_camera frlr_prefix="front" lrc_prefix="left">
+    <origin xyz="-0.04 0.12 1.3" rpy="0 0.087 0"/>
+  </xacro:sekonix_camera>
+  <xacro:sekonix_camera frlr_prefix="front" lrc_prefix="right">
+    <origin xyz="-0.04 -0.12 1.3" rpy="0 0.087 0"/>
+  </xacro:sekonix_camera>
+  <xacro:sekonix_camera frlr_prefix="front" lrc_prefix="center">
+    <origin xyz="-0.04 0 1.3" rpy="0 0.087 0"/>
+  </xacro:sekonix_camera>
+  <xacro:sekonix_camera frlr_prefix="rear" lrc_prefix="center">
+    <origin xyz="-1.26 0 1.28" rpy="0 0.2618 3.14"/>
+  </xacro:sekonix_camera>
+  <xacro:sekonix_camera frlr_prefix="right" lrc_prefix="forward">
+    <origin xyz="-0.95 -0.42 1.2" rpy="0 0.244 -1.12"/>
+  </xacro:sekonix_camera>
+  <xacro:sekonix_camera frlr_prefix="right" lrc_prefix="rearward">
+    <origin xyz="-1.05 -0.42 1.2" rpy="0 0.244 -2.18"/>
+  </xacro:sekonix_camera>
+  <xacro:sekonix_camera frlr_prefix="left" lrc_prefix="forward">
+    <origin xyz="-0.95 0.4 1.2" rpy="0 0.2967 1.12"/>
+  </xacro:sekonix_camera>
+  <xacro:sekonix_camera frlr_prefix="left" lrc_prefix="rearward">
+    <origin xyz="-1.05 0.39 1.2" rpy="0 0.2967 2.18"/>
+  </xacro:sekonix_camera>
   <gazebo>
     <plugin name="sd_control" filename="libSdControlPlugin.so">
+      <chassis>base_link</chassis>
+      <front_left_wheel>front_left_wheel_joint</front_left_wheel>
+      <front_right_wheel>front_right_wheel_joint</front_right_wheel>
+      <front_left_wheel_steering>front_left_steer_joint</front_left_wheel_steering>
+      <front_right_wheel_steering>front_right_steer_joint</front_right_wheel_steering>
+      <back_left_wheel>rear_left_wheel_joint</back_left_wheel>
+      <back_right_wheel>rear_right_wheel_joint</back_right_wheel>
     </plugin>
   </gazebo>
-    <!-- ***************** -->
-    <!-- Imported elements -->
-    <!-- ***************** -->
-    <xacro:include filename="$(find sd_description)/urdf/bases/sd_twizy_body.urdf.xacro" />
-    <xacro:include filename="$(find sd_description)/urdf/wheels/sd_twizy_suspension.urdf.xacro" />
-    <xacro:include filename="$(find sd_description)/urdf/sensors/VLP-16.urdf.xacro"/>
-    <xacro:include filename="$(find sd_description)/urdf/sensors/cameras.urdf.xacro"/>
-    <!-- *************** -->
-    <!-- Robots Elements -->
-    <!-- *************** -->
-    <xacro:sd_twizy_base name="sd_twizy"/>
-    <xacro:ros_control/>
-    <xacro:RL_wheel/>
-    <xacro:RR_wheel/>
-    <xacro:FL_wheel/>
-    <xacro:FR_wheel/>
-    <!-- Sensors -->
-    <xacro:VLP-16  parent="base_link" name="velodyne" topic="/points_raw" hz="10" samples="1875">
-        <origin xyz="-0.681 0 1.445" rpy="0 -${1.5*M_PI/180.0} 0"/>
-    </xacro:VLP-16>
-    <xacro:sekonix_camera frlr_prefix="front" lrc_prefix="left">
-        <origin xyz="-0.04 0.12 1.3" rpy="0 0.087 0"/>
-    </xacro:sekonix_camera>
-    <xacro:sekonix_camera frlr_prefix="front" lrc_prefix="right">
-        <origin xyz="-0.04 -0.12 1.3" rpy="0 0.087 0"/>
-    </xacro:sekonix_camera>
-    <xacro:sekonix_camera frlr_prefix="front" lrc_prefix="center">
-        <origin xyz="-0.04 0 1.3" rpy="0 0.087 0"/>
-    </xacro:sekonix_camera>
-    <xacro:sekonix_camera frlr_prefix="rear" lrc_prefix="center">
-        <origin xyz="-1.26 0 1.28" rpy="0 0.2618 3.14"/>
-    </xacro:sekonix_camera>
-    <xacro:sekonix_camera frlr_prefix="right" lrc_prefix="forward">
-        <origin xyz="-0.95 -0.42 1.2" rpy="0 0.244 -1.12"/>
-    </xacro:sekonix_camera>
-    <xacro:sekonix_camera frlr_prefix="right" lrc_prefix="rearward">
-        <origin xyz="-1.05 -0.42 1.2" rpy="0 0.244 -2.18"/>
-    </xacro:sekonix_camera>
-    <xacro:sekonix_camera frlr_prefix="left" lrc_prefix="forward">
-        <origin xyz="-0.95 0.4 1.2" rpy="0 0.2967 1.12"/>
-    </xacro:sekonix_camera>
-    <xacro:sekonix_camera frlr_prefix="left" lrc_prefix="rearward">
-        <origin xyz="-1.05 0.39 1.2" rpy="0 0.2967 2.18"/>
-    </xacro:sekonix_camera>
 </robot>

File: streetdrone_model/sd_description/urdf/sensors/cameras.urdf.xacro (robot description, xacro)
@@ -1,96 +1,96 @@
 <?xml version="1.0"?>
 <!--
-  Copyright (c) 2019 StreetDrone Limited
-  Author:  Efimia Panagiotaki
-  All rights reserved
+Copyright (c) 2019 StreetDrone Limited
+Author:  Efimia Panagiotaki
+All rights reserved
 -->
 <robot xmlns:xacro="http://www.ros.org/wiki/xacro" name="sekonix_camera">
-    <xacro:macro name="sekonix_camera" params="frlr_prefix lrc_prefix *origin">
-        <joint name="${frlr_prefix}_${lrc_prefix}_camera_joint" type="fixed">
-            <axis xyz="0 1 0" />
-            <xacro:insert_block name="origin"/>
-            <parent link="base_link"/>
-            <child link="${frlr_prefix}_${lrc_prefix}_camera_link"/>
-        </joint>
-        <!-- Camera -->
-        <link name="${frlr_prefix}_${lrc_prefix}_camera_link">
-            <collision>
-                <origin xyz="0 0 0" rpy="0 0 0"/>
-                <geometry>
-                    <box size="0.026 0.026 0.0203"/>
-                </geometry>
-            </collision>
-            <visual>
-                <origin xyz="0 0 0" rpy="0 0 0"/>
-                <geometry>
-                    <box size="0.026 0.026 0.0203"/>
-                </geometry>
-                <material name="red"/>
-            </visual>
-            <inertial>
-                <mass value="1e-5" />
-                <origin xyz="0 0 0" rpy="0 0 0"/>
-                <inertia ixx="1e-6" ixy="0" ixz="0" iyy="1e-6" iyz="0" izz="1e-6" />
-            </inertial>
-        </link>
-        <!-- generate an optical frame http://www.ros.org/reps/rep-0103.html#suffix-frames
-            so that ros and opencv can operate on the camera frame correctly -->
-        <joint name="${frlr_prefix}_${lrc_prefix}_camera_optical_joint" type="fixed">
-            <!-- these values have to be these values otherwise the gazebo camera image
-                won't be aligned properly with the frame it is supposedly originating from -->
-            <origin xyz="0 0 0" rpy="${-pi/2} 0 ${-pi/2}"/>
-            <parent link="${frlr_prefix}_${lrc_prefix}_camera_link"/>
-            <child link="${frlr_prefix}_${lrc_prefix}_camera_link_optical"/>
-        </joint>
-        <link name="${frlr_prefix}_${lrc_prefix}_camera_link_optical"/>
-        <gazebo reference="${frlr_prefix}_${lrc_prefix}_camera_link">
-            <mu1>0.2</mu1>
-            <mu2>0.2</mu2>
-            <material>Gazebo/Red</material>
-            <sensor type="camera" name="${frlr_prefix}_${lrc_prefix}_camera">
-                <update_rate>30.0</update_rate>
-                <camera name="head">
-                    <horizontal_fov>2.09</horizontal_fov>
-                    <image>
-                        <width>1928</width>
-                        <height>1208</height>
-                        <format>R8G8B8</format>
-                    </image>
-                    <clip>
-                        <near>0.1</near>
-                        <far>30</far>
-                    </clip>
-                    <noise>
-                        <type>gaussian</type>
-                        <!-- Noise is sampled independently per pixel on each frame.
-                             That pixel's noise value is added to each of its color
-                             channels, which at that point lie in the range [0,1]. -->
-                        <mean>0.0</mean>
-                        <stddev>0.007</stddev>
-                    </noise>
-                </camera>
-                <plugin name="${frlr_prefix}_${lrc_prefix}_camera_controller" filename="libgazebo_ros_camera.so">
-                    <alwaysOn>true</alwaysOn>
-                    <updateRate>0.0</updateRate>
-                    <cameraName>sd_twizy/${frlr_prefix}_${lrc_prefix}_camera</cameraName>
-                    <imageTopicName>image_raw</imageTopicName>
-                    <cameraInfoTopicName>camera_info</cameraInfoTopicName>
-                    <frameName>${frlr_prefix}_${lrc_prefix}_camera_link_optical</frameName>
-                    <!-- setting hackBaseline to anything but 0.0 will cause a misalignment
-                        between the gazebo sensor image and the frame it is supposed to
-                        be attached to -->
-                    <hackBaseline>0.0</hackBaseline>
-                    <distortionK1>0.0</distortionK1>
-                    <distortionK2>0.0</distortionK2>
-                    <distortionK3>0.0</distortionK3>
-                    <distortionT1>0.0</distortionT1>
-                    <distortionT2>0.0</distortionT2>
-                    <CxPrime>0</CxPrime>
-                    <Cx>0.0</Cx>
-                    <Cy>0.0</Cy>
-                    <focalLength>0.0</focalLength>
-                </plugin>
-            </sensor>
-        </gazebo>
-    </xacro:macro>
+  <xacro:macro name="sekonix_camera" params="frlr_prefix lrc_prefix *origin">
+    <joint name="${frlr_prefix}_${lrc_prefix}_camera_joint" type="fixed">
+      <axis xyz="0 1 0" />
+      <xacro:insert_block name="origin"/>
+      <parent link="chassis"/>
+      <child link="${frlr_prefix}_${lrc_prefix}_camera_link"/>
+    </joint>
+    <!-- Camera -->
+    <link name="${frlr_prefix}_${lrc_prefix}_camera_link">
+      <collision>
+        <origin xyz="0 0 0" rpy="0 0 0"/>
+        <geometry>
+          <box size="0.026 0.026 0.0203"/>
+        </geometry>
+      </collision>
+      <visual>
+        <origin xyz="0 0 0" rpy="0 0 0"/>
+        <geometry>
+          <box size="0.026 0.026 0.0203"/>
+        </geometry>
+        <material name="red"/>
+      </visual>
+      <inertial>
+        <mass value="1e-5" />
+        <origin xyz="0 0 0" rpy="0 0 0"/>
+        <inertia ixx="1e-6" ixy="0" ixz="0" iyy="1e-6" iyz="0" izz="1e-6" />
+      </inertial>
+    </link>
+    <!-- generate an optical frame http://www.ros.org/reps/rep-0103.html#suffix-frames
+         so that ros and opencv can operate on the camera frame correctly -->
+    <joint name="${frlr_prefix}_${lrc_prefix}_camera_optical_joint" type="fixed">
+      <!-- these values have to be these values otherwise the gazebo camera image
+           won't be aligned properly with the frame it is supposedly originating from -->
+      <origin xyz="0 0 0" rpy="${-pi/2} 0 ${-pi/2}"/>
+      <parent link="${frlr_prefix}_${lrc_prefix}_camera_link"/>
+      <child link="${frlr_prefix}_${lrc_prefix}_camera_link_optical"/>
+    </joint>
+    <link name="${frlr_prefix}_${lrc_prefix}_camera_link_optical"/>
+    <gazebo reference="${frlr_prefix}_${lrc_prefix}_camera_link">
+      <mu1>0.2</mu1>
+      <mu2>0.2</mu2>
+      <material>Gazebo/Red</material>
+      <sensor type="camera" name="${frlr_prefix}_${lrc_prefix}_camera">
+        <update_rate>30.0</update_rate>
+        <camera name="head">
+          <horizontal_fov>2.09</horizontal_fov>
+          <image>
+            <width>1928</width>
+            <height>1208</height>
+            <format>R8G8B8</format>
+          </image>
+          <clip>
+            <near>0.1</near>
+            <far>30</far>
+          </clip>
+          <noise>
+            <type>gaussian</type>
+            <!-- Noise is sampled independently per pixel on each frame.
+                 That pixel's noise value is added to each of its color
+                 channels, which at that point lie in the range [0,1]. -->
+            <mean>0.0</mean>
+            <stddev>0.007</stddev>
+          </noise>
+        </camera>
+        <plugin name="${frlr_prefix}_${lrc_prefix}_camera_controller" filename="libgazebo_ros_camera.so">
+          <alwaysOn>true</alwaysOn>
+          <updateRate>0.0</updateRate>
+          <cameraName>sd_twizy/${frlr_prefix}_${lrc_prefix}_camera</cameraName>
+          <imageTopicName>image_raw</imageTopicName>
+          <cameraInfoTopicName>camera_info</cameraInfoTopicName>
+          <frameName>${frlr_prefix}_${lrc_prefix}_camera_link_optical</frameName>
+          <!-- setting hackBaseline to anything but 0.0 will cause a misalignment
+               between the gazebo sensor image and the frame it is supposed to
+               be attached to -->
+          <hackBaseline>0.0</hackBaseline>
+          <distortionK1>0.0</distortionK1>
+          <distortionK2>0.0</distortionK2>
+          <distortionK3>0.0</distortionK3>
+          <distortionT1>0.0</distortionT1>
+          <distortionT2>0.0</distortionT2>
+          <CxPrime>0</CxPrime>
+          <Cx>0.0</Cx>
+          <Cy>0.0</Cy>
+          <focalLength>0.0</focalLength>
+        </plugin>
+      </sensor>
+    </gazebo>
+  </xacro:macro>
 </robot>
