Commit message: Torque based control - ROS Melodic release
* Remove files generated from source

* Disable front wheel drive

* Ensure launch files and worlds are installed

* Initial functionality of control plugin loaded from model

* Cleanup URDF files and make links and joints resolvable in plugin

* Steering, throttle and breaking implemented

Max speed and torque are set based on engine and gearbox specs,
source:

https://www.cdn.renault.com/content/dam/Renault/MY/electric-vehicles/twizy/b09e-twizy/b09e-phase1/product-brochures/Renault-Twizy-Pricelist-2017.pdf

* Add sd_control_msgs package

* Teleop node to drive SD model with a joystick

* Clean up launch file and add one for teleop

* Remove old control node

* Remove ros_control plugin and add joint state pub plugin to URDF

* Determine odometry in local frame and publish on topic

This assumes operation on a flat 2D plane

* Add node to control SD with Autoware ctrl_cmd output

* Add launch file for PID and sd_autoware node needed to work with ctrl_cmd

* Rename bringup package and cleanup some files

* Update and clean up launch files

to spawn model at right height, more informative naming and reduce
duplication

* Fix using base link as fixed frame in rviz conf

* Fix too many slashes in file paths

* Ensure launch file with joint publisher is included in launch files

* Update dependencies

* Add CATKIN_IGNORE file to not automatically build sd_autoware package

* Update main readme file

* Fix source path in rosdep install command

* Do not run Gazebo in verbose mode

* Add missing dependency on joy package

* Update steps: don't install gazebo manually, checkout right branch

All dependencies including Gazebo are installed using `rosdep`

* Add know issues

* Expand on how to use sd_twizy_spawn.launch

Co-authored-by: Sander van Dijk <sander@parkopedia.com>

File: streetdrone_model/sd_description/urdf/bases/sd_twizy_body.gazebo.xacro (robot description, xacro)
@@ -1,30 +1,11 @@
 <?xml version="1.0"?>
 <!--
-  Copyright (c) 2019 StreetDrone Limited
-  Author:  Efimia Panagiotaki
-  All rights reserved
+Copyright (c) 2019 StreetDrone Limited
+Author:  Efimia Panagiotaki
+All rights reserved
 -->
 <robot xmlns:xacro="http://www.ros.org/wiki/xacro">
-   <gazebo>
-        <plugin name="p3d" filename="libgazebo_ros_p3d.so">
-            <bodyName>base_link</bodyName>
-            <topicName>base_pose_ground_truth</topicName>
-            <frameName>map</frameName>
-            <updateRate>100.0</updateRate>
-        </plugin>
-    </gazebo>
-  <!-- ros control plugin -->
-  <xacro:macro name="ros_control">
-    <gazebo>
-            <plugin name="gazebo_ros_control" filename="libgazebo_ros_control.so">
-                <robotNamespace>/sd_twizy</robotNamespace>
-                <controlPeriod>0.001</controlPeriod>
-                <robotSimType>gazebo_ros_control/DefaultRobotHWSim</robotSimType>
-                <legacyModeNS>true</legacyModeNS>
-            </plugin>
-        </gazebo>
-    </xacro:macro>
-    <gazebo reference="base_link">-->
-        <material>Gazebo/Green</material>
-    </gazebo>
+  <gazebo reference="chassis">
+    <material>Gazebo/Green</material>
+  </gazebo>
 </robot>

File: streetdrone_model/sd_description/urdf/bases/sd_twizy_body.urdf.xacro (robot description, xacro)
@@ -1,48 +1,49 @@
 <?xml version="1.0"?>
 <!--
-  Copyright (c) 2019 StreetDrone Limited
-  Author:  Efimia Panagiotaki
-  All rights reserved
+Copyright (c) 2019 StreetDrone Limited
+Author:  Efimia Panagiotaki
+All rights reserved
 -->
 <robot name="sd_twizy" xmlns:xacro="http://www.ros.org/wiki/xacro">
-    <xacro:include filename="$(find sd_description)/urdf/bases/sd_twizy_body.gazebo.xacro" />
-    <xacro:macro name="sd_twizy_base" params="name">
-        <xacro:property name="depth" value="2.352"/>
-        <xacro:property name="height" value="1.7"/>
-        <xacro:property name="width" value="1.431"/>
-        <xacro:property name="base_mass" value="435"/>
-        <xacro:property name="clearance" value="0.281"/>
-        <link name="vehicle_base">
-            <visual>
-                <origin xyz="0 0 0" rpy="0 0 0" />
-                <geometry>
-                    <box size="0.001 0.001 0.001" />
-                </geometry>
-            </visual>
-        </link>
-        <joint name="vehicle_base_joint" type="fixed">
-            <origin xyz="0 0 ${clearance}" rpy="0 0 0"/>
-            <parent link="vehicle_base"/>
-            <child link="base_link"/>
-        </joint>
-        <link name="base_link">
-            <inertial>
-                <mass value="${base_mass}"/>
-                <origin xyz="0 0 0"/>
-                <inertia ixx="243.175" ixy="0" ixz="0" iyy="430.166" iyz="0" izz="430.166"/>
-            </inertial>
-            <visual>
-                <origin xyz="0 0 0" rpy="0 0 1.57079632679"/>
-                <geometry>
-                    <mesh filename="file:///$(find sd_description)/meshes/SDTwizy.stl" scale="0.01 0.01 0.01"/>
-		</geometry>
-            </visual>
-            <collision>
-                <origin xyz="0 0 0" rpy="0 0 1.57079632679"/>
-                <geometry>
-                    <mesh filename="file:///$(find sd_description)/meshes/SDTwizy_collision.stl" scale="0.01 0.01 0.01"/>
-		</geometry>
-            </collision>
-        </link>
-    </xacro:macro>
+  <xacro:include filename="$(find sd_description)/urdf/bases/sd_twizy_body.gazebo.xacro" />
+  <xacro:macro name="sd_twizy_base" params="name">
+    <xacro:property name="depth" value="2.352"/>
+    <xacro:property name="height" value="1.7"/>
+    <xacro:property name="width" value="1.431"/>
+    <xacro:property name="base_mass" value="435"/>
+    <xacro:property name="clearance" value="0.281"/>
+    <xacro:property name = "wheelbase" value="1.686"/>
+    <link name="base_link">
+      <visual>
+        <origin xyz="0 0 0" rpy="0 0 0" />
+        <geometry>
+          <box size="0.001 0.001 0.001" />
+        </geometry>
+      </visual>
+    </link>
+    <joint name="chassis_joint" type="fixed">
+      <origin xyz="${wheelbase / 2} 0 0" rpy="0 0 0"/>
+      <parent link="base_link"/>
+      <child link="chassis"/>
+    </joint>
+    <link name="chassis">
+      <inertial>
+        <mass value="${base_mass}"/>
+        <origin xyz="0 0 0"/>
+        <inertia ixx="243.175" ixy="0" ixz="0" iyy="430.166" iyz="0" izz="430.166"/>
+      </inertial>
+      <visual>
+        <origin xyz="0 0 0" rpy="0 0 1.57079632679"/>
+        <geometry>
+          <mesh filename="file://$(find sd_description)/meshes/SDTwizy.stl" scale="0.01 0.01 0.01"/>
+        </geometry>
+      </visual>
+      <collision>
+        <origin xyz="0 0 0" rpy="0 0 1.57079632679"/>
+        <geometry>
+          <mesh filename="file://$(find sd_description)/meshes/SDTwizy_collision.stl" scale="0.01 0.01 0.01"/>
+        </geometry>
+      </collision>
+    </link>
+  </xacro:macro>
 </robot>

File: streetdrone_model/sd_description/urdf/sd_twizy.urdf.xacro (robot description, xacro)
@@ -1,52 +1,89 @@
 <?xml version="1.0"?>
 <!--
-  Copyright (c) 2019 StreetDrone Limited
-  Author:  Efimia Panagiotaki
-  All rights reserved
+Copyright (c) 2019 StreetDrone Limited
+Author:  Efimia Panagiotaki
+All rights reserved
 -->
 <robot name="sd_twizy" xmlns:xacro="http://www.ros.org/wiki/xacro">
-    <!-- ***************** -->
-    <!-- Imported elements -->
-    <!-- ***************** -->
-    <xacro:include filename="$(find sd_description)/urdf/bases/sd_twizy_body.urdf.xacro" />
-    <xacro:include filename="$(find sd_description)/urdf/wheels/sd_twizy_suspension.urdf.xacro" />
-    <xacro:include filename="$(find sd_description)/urdf/sensors/VLP-16.urdf.xacro"/>
-    <xacro:include filename="$(find sd_description)/urdf/sensors/cameras.urdf.xacro"/>
-    <!-- *************** -->
-    <!-- Robots Elements -->
-    <!-- *************** -->
-    <xacro:sd_twizy_base name="sd_twizy"/>
-    <xacro:ros_control/>
-    <xacro:RL_wheel/>
-    <xacro:RR_wheel/>
-    <xacro:FL_wheel/>
-    <xacro:FR_wheel/>
-    <!-- Sensors -->
-    <xacro:VLP-16  parent="base_link" name="velodyne" topic="/points_raw" hz="10" samples="1875">
-        <origin xyz="-0.681 0 1.445" rpy="0 -${1.5*M_PI/180.0} 0"/>
-    </xacro:VLP-16>
-    <xacro:sekonix_camera frlr_prefix="front" lrc_prefix="left">
-        <origin xyz="-0.04 0.12 1.3" rpy="0 0.087 0"/>
-    </xacro:sekonix_camera>
-    <xacro:sekonix_camera frlr_prefix="front" lrc_prefix="right">
-        <origin xyz="-0.04 -0.12 1.3" rpy="0 0.087 0"/>
-    </xacro:sekonix_camera>
-    <xacro:sekonix_camera frlr_prefix="front" lrc_prefix="center">
-        <origin xyz="-0.04 0 1.3" rpy="0 0.087 0"/>
-    </xacro:sekonix_camera>
-    <xacro:sekonix_camera frlr_prefix="rear" lrc_prefix="center">
-        <origin xyz="-1.26 0 1.28" rpy="0 0.2618 3.14"/>
-    </xacro:sekonix_camera>
-    <xacro:sekonix_camera frlr_prefix="right" lrc_prefix="forward">
-        <origin xyz="-0.95 -0.42 1.2" rpy="0 0.244 -1.12"/>
-    </xacro:sekonix_camera>
-    <xacro:sekonix_camera frlr_prefix="right" lrc_prefix="rearward">
-        <origin xyz="-1.05 -0.42 1.2" rpy="0 0.244 -2.18"/>
-    </xacro:sekonix_camera>
-    <xacro:sekonix_camera frlr_prefix="left" lrc_prefix="forward">
-        <origin xyz="-0.95 0.4 1.2" rpy="0 0.2967 1.12"/>
-    </xacro:sekonix_camera>
-    <xacro:sekonix_camera frlr_prefix="left" lrc_prefix="rearward">
-        <origin xyz="-1.05 0.39 1.2" rpy="0 0.2967 2.18"/>
-    </xacro:sekonix_camera>
+  <!-- ***************** -->
+  <!-- Imported elements -->
+  <!-- ***************** -->
+  <xacro:include filename="$(find sd_description)/urdf/bases/sd_twizy_body.urdf.xacro" />
+  <xacro:include filename="$(find sd_description)/urdf/wheels/sd_twizy_suspension.urdf.xacro" />
+  <xacro:include filename="$(find sd_description)/urdf/sensors/VLP-16.urdf.xacro"/>
+  <xacro:include filename="$(find sd_description)/urdf/sensors/cameras.urdf.xacro"/>
+  <!-- *************** -->
+  <!-- Robots Elements -->
+  <!-- *************** -->
+  <xacro:sd_twizy_base name="sd_twizy"/>
+  <xacro:RL_wheel/>
+  <xacro:RR_wheel/>
+  <xacro:FL_wheel/>
+  <xacro:FR_wheel/>
+  <!-- Sensors -->
+  <xacro:VLP-16  parent="chassis" name="velodyne" topic="/points_raw" hz="10" samples="1875">
+    <origin xyz="-0.681 0 1.445" rpy="0 -${1.5*M_PI/180.0} 0"/>
+  </xacro:VLP-16>
+  <xacro:sekonix_camera frlr_prefix="front" lrc_prefix="left">
+    <origin xyz="-0.04 0.12 1.3" rpy="0 0.087 0"/>
+  </xacro:sekonix_camera>
+  <xacro:sekonix_camera frlr_prefix="front" lrc_prefix="right">
+    <origin xyz="-0.04 -0.12 1.3" rpy="0 0.087 0"/>
+  </xacro:sekonix_camera>
+  <xacro:sekonix_camera frlr_prefix="front" lrc_prefix="center">
+    <origin xyz="-0.04 0 1.3" rpy="0 0.087 0"/>
+  </xacro:sekonix_camera>
+  <xacro:sekonix_camera frlr_prefix="rear" lrc_prefix="center">
+    <origin xyz="-1.26 0 1.28" rpy="0 0.2618 3.14"/>
+  </xacro:sekonix_camera>
+  <xacro:sekonix_camera frlr_prefix="right" lrc_prefix="forward">
+    <origin xyz="-0.95 -0.42 1.2" rpy="0 0.244 -1.12"/>
+  </xacro:sekonix_camera>
+  <xacro:sekonix_camera frlr_prefix="right" lrc_prefix="rearward">
+    <origin xyz="-1.05 -0.42 1.2" rpy="0 0.244 -2.18"/>
+  </xacro:sekonix_camera>
+  <xacro:sekonix_camera frlr_prefix="left" lrc_prefix="forward">
+    <origin xyz="-0.95 0.4 1.2" rpy="0 0.2967 1.12"/>
+  </xacro:sekonix_camera>
+  <xacro:sekonix_camera frlr_prefix="left" lrc_prefix="rearward">
+    <origin xyz="-1.05 0.39 1.2" rpy="0 0.2967 2.18"/>
+  </xacro:sekonix_camera>
+  <gazebo>
+    <plugin name="sd_control" filename="libSdControlPlugin.so">
+      <chassis>base_link</chassis>
+      <front_left_wheel>front_left_wheel_joint</front_left_wheel>
+      <front_right_wheel>front_right_wheel_joint</front_right_wheel>
+      <front_left_wheel_steering>front_left_steer_joint</front_left_wheel_steering>
+      <front_right_wheel_steering>front_right_steer_joint</front_right_wheel_steering>
+      <back_left_wheel>rear_left_wheel_joint</back_left_wheel>
+      <back_right_wheel>rear_right_wheel_joint</back_right_wheel>
+      <fl_wheel_steering_p_gain>1e4</fl_wheel_steering_p_gain>
+      <fr_wheel_steering_p_gain>1e4</fr_wheel_steering_p_gain>
+      <fl_wheel_steering_i_gain>0</fl_wheel_steering_i_gain>
+      <fr_wheel_steering_i_gain>0</fr_wheel_steering_i_gain>
+      <fl_wheel_steering_d_gain>3e2</fl_wheel_steering_d_gain>
+      <fr_wheel_steering_d_gain>3e2</fr_wheel_steering_d_gain>
+      <max_speed>22</max_speed>
+      <max_torque>250</max_torque>
+      <front_brake_torque>260</front_brake_torque>
+      <back_brake_torque>260</back_brake_torque>
+      <chassis_aero_force_gain>0.63045</chassis_aero_force_gain>
+    </plugin>
+  </gazebo>
+  <gazebo>
+    <plugin name="p3d" filename="libgazebo_ros_p3d.so">
+      <bodyName>base_link</bodyName>
+      <topicName>base_pose_ground_truth</topicName>
+      <frameName>map</frameName>
+      <updateRate>100.0</updateRate>
+    </plugin>
+  </gazebo>
+  <gazebo>
+    <plugin name="joint_state_publisher" filename="libgazebo_ros_joint_state_publisher.so">
+      <robotNamespace>/sd_twizy</robotNamespace>
+      <jointName>front_left_wheel_joint, front_right_wheel_joint, front_left_steer_joint, front_right_steer_joint, rear_left_wheel_joint, rear_right_wheel_joint</jointName>
+      <updateRate>100.0</updateRate>
+      <alwaysOn>true</alwaysOn>
+    </plugin>
+  </gazebo>
 </robot>
